File: pcb/p4_joint.brd (EAGLE design)
At the start: 50 x 50 mm, 14 parts

Commit message: pcb(p4_joint): avance rev B (WIP, sin terminar)
Trabajo en curso del diseno: rele G5V-2, diodo SS14, transistores SOT-23 y
conectores 1X04 anadidos al esquema y la placa. Falta acabar el enrutado y la
revision final; se commitea para poder cortar el release v1.0.10 del firmware
con el arbol limpio.

Co-Authored-By: Claude Opus 4.8 (1M context) <noreply@anthropic.com>
Parts:
- added D1, D3: SS14, p4_joint_add:SMA
- added JP6: (no value), pinhead:1X04
- added JP7, JP8, JP9: (no value), pinhead:1X02
- added K1: JS1APF-B-12V, p4_joint_add:JS_RELAY_1A
- added K2: G5V-2, relay:G5V-2
- added Q1, Q2: 2N7002, zetex:SOT-23
- added R2, R5: 10k, eagle-ltspice:R0805
- added R6, R7: 100, eagle-ltspice:R0805
- added RELE_OUT, RELE_OUT1, RELE_OUT2, RELE_OUT3: (no value), con-molex:KK-156-2
- JP1: value (none) -> DS18B20_IN; device pinhead:1X02 -> pinhead:1X03
- JP3: value DS18B20_1 -> DS18B20_3
- U$1: value IRLR7843 -> LR7843
- moved FAN_OUT 41.1 mm to (26.7, 82.5)
- moved D2 39.9 mm to (26.7, 73.7)
- moved R3 34.3 mm to (21.6, 49.5)
- moved R4 33.9 mm to (26.7, 50.4)
- moved U$1 33.1 mm to (25.4, 59.7)
- moved JP2 29.3 mm to (8.89, 39.4)
- moved JP1 28.5 mm to (8.89, 31.8)
- moved JP4 21.7 mm to (8.89, 48.3)
- moved JP5 19.2 mm to (8.89, 54.6)
- moved R1 19.2 mm to (8.89, 59.7)
- moved C3 14.0 mm to (38.1, 35.6)
- moved C2 12.7 mm to (36.8, 29.2)
- moved DC_IN 10.2 mm to (36.8, 17.8)
- moved JP3 4.58 mm to (8.89, 15.2)
Connections:
- removed net DATA_DS18B20: JP2.3, JP3.3, JP4.3, JP5.3, R1.1
- new net N$10: K2.16, Q1.1
- new net N$11: Q1.3, R6.2
- new net N$12: JP6.4, R6.1
- new net N$13: JP6.3, R7.1
- new net N$14: Q2.3, R2.2, R7.2
- new net N$15: D3.A
- new net N$16: JP8.2, K2.4, RELE_OUT3.1
- new net N$17: JP7.1, K1.3
- new net N$18: K1.1, RELE_OUT1.2
- new net N$19: JP9.1, RELE_OUT2.2
- new net N$20: JP9.2, K2.13
- new net N$5: R5.2
- new net N$9: D1.A, K1.5, Q2.1
- net +3V3: now also JP1.1
- net 12V: now also D1.C, D3.C, JP7.2, K1.2, K2.1, RELE_OUT1.1
- net GND: now also JP1.2, JP1.3, JP2.3, JP3.3, JP4.3, JP5.3, Q2.2, R1.1, R2.1
- net N$6: no longer JP1.1
Routing:
- net 12V: track 36.9 -> 70.0 mm
- net DATA_DS18B20: track 31.9 -> 0.00 mm
- net +3V3: track 31.9 -> 44.6 mm
- net GND: track 2.06 -> 8.96 mm
- net N$6: track 6.89 -> 0.00 mm
- net N$2: track 14.2 -> 20.8 mm
- net N$3: track 11.7 -> 9.30 mm
Other:
- board size 50 x 50 mm -> 100 x 100 mm
