File: pcb/p4_joint.brd (EAGLE design)
At the start: 100 x 100 mm, 32 parts, among them K1 JS1APF-B-12V, K2 G5V-2, Q1 2N7002, Q2 2N7002

Commit message: pcb: reubicar el conector RELE_OUT2 y añadir JP9/RELE_OUT3 con sus señales
Parts:
- moved RELE_OUT2 54.3 mm to (87.6, 24.1)
Changed lines of the file:
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@@
 <attribute name="VALUE" x="74.22" y="79.06" size="1" layer="27" font="vector" rot="R270"/>
 </element>
-<element name="RELE_OUT2" library="con-molex" library_urn="urn:adsk.eagle:library:165" package="KK-156-2" package3d_urn="urn:adsk.eagle:package:8078800/1" value="" x="77.47" y="-29.21" smashed="yes">
-<attribute name="MF" value="MOLEX" x="77.47" y="-26.67" size="1.778" layer="27" display="off"/>
-<attribute name="MPN" value="" x="77.47" y="-26.67" size="1.778" layer="27" display="off"/>
-<attribute name="NAME" x="72.99" y="-33.655" size="1.27" layer="25" rot="R90"/>
-<attribute name="OC_FARNELL" value="unknown" x="77.47" y="-26.67" size="1.778" layer="27" display="off"/>
-<attribute name="OC_NEWARK" value="unknown" x="77.47" y="-26.67" size="1.778" layer="27" display="off"/>
-<attribute name="POPULARITY" value="10" x="77.47" y="-26.67" size="1.778" layer="27" display="off"/>
-<attribute name="VALUE" x="83.22" y="-33.655" size="1.27" layer="27" rot="R90"/>
+<element name="RELE_OUT2" library="con-molex" library_urn="urn:adsk.eagle:library:165" package="KK-156-2" package3d_urn="urn:adsk.eagle:package:8078800/1" value="" x="87.63" y="24.13" smashed="yes">
+<attribute name="MF" value="MOLEX" x="87.63" y="26.67" size="1.778" layer="27" display="off"/>
+<attribute name="MPN" value="" x="87.63" y="26.67" size="1.778" layer="27" display="off"/>
+<attribute name="NAME" x="83.15" y="19.685" size="1.27" layer="25" rot="R90"/>
+<attribute name="OC_FARNELL" value="unknown" x="87.63" y="26.67" size="1.778" layer="27" display="off"/>
+<attribute name="OC_NEWARK" value="unknown" x="87.63" y="26.67" size="1.778" layer="27" display="off"/>
+<attribute name="POPULARITY" value="10" x="87.63" y="26.67" size="1.778" layer="27" display="off"/>
+<attribute name="VALUE" x="93.38" y="19.685" size="1.27" layer="27" rot="R90"/>
 </element>
 <element name="JP3" library="pinhead" library_urn="urn:adsk.eagle:library:325" package="1X03" package3d_urn="urn:adsk.eagle:package:22458/2" value="DS18B20_3" x="8.89" y="15.24" smashed="yes">
@@
 <contactref element="JP9" pad="1"/>
 <contactref element="RELE_OUT2" pad="2"/>
-<wire x1="79.45" y1="-29.21" x2="1.27" y2="-142.24" width="0" layer="19" extent="1-1"/>
+<wire x1="89.61" y1="24.13" x2="1.27" y2="-142.24" width="0" layer="19" extent="1-1"/>
 </signal>
 <signal name="N$20">

Commit message: fix(ne185): filtrar el baile del nivel de agua limpia segun si el motor esta en marcha
Parts:
- added JP10: (no value), pinhead:1X04
Connections:
- removed net +3V3: JP1.1, JP2.1, JP3.1, JP4.1, JP5.1, R1.2
- removed net GND: C2.-, C3.2, DC_IN.2, JP1.2, JP1.3, JP2.2, JP2.3, JP3.2, JP3.3, JP4.2, JP4.3, JP5.2, JP5.3, Q2.2, R1.1, R2.1, R4.2, U$1.2
- removed net N$10: K2.16, Q1.1
- removed net N$13: JP6.3, R7.1
- removed net N$14: Q2.3, R2.2, R7.2
- removed net N$15: D3.A
- removed net N$16: JP8.2, K2.4, RELE_OUT3.1
- removed net N$17: JP7.1, K1.3
- removed net N$18: K1.1, RELE_OUT1.2
- removed net N$19: JP9.1, RELE_OUT2.2
- removed net N$20: JP9.2, K2.13
- removed net N$3: R3.1, R4.1, U$1.1
- removed net N$9: D1.A, K1.5, Q2.1
- new net N$21: JP1.2, JP2.2, JP3.2, JP4.2, JP5.2
- new net N$22: JP1.1, JP2.1, JP3.1, JP4.1, JP5.1
- net 12V: no longer C2.+, C3.1, D1.C, D2.C, D3.C, DC_IN.1, FAN_OUT.1, JP7.2, K1.2, RELE_OUT1.1
- net N$11: no longer Q1.3
- net N$12: now also K1.5; no longer JP6.4, R6.1
- net N$2: now also JP1.3, JP2.3, JP3.3, JP4.3, JP5.3; no longer D2.A, FAN_OUT.2, U$1.3
- net N$6: now also Q2.3; no longer R3.2
Routing:
- net 12V: track 70.0 -> 0.00 mm
- net +3V3: track 44.6 -> 0.00 mm
- net N$2: track 20.8 -> 0.00 mm
- net N$3: track 9.30 -> 0.00 mm
- net GND: track 8.96 -> 0.00 mm
Changed lines of the file:
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@@
 <attribute name="VALUE" x="12.1" y="-154.305" size="1.27" layer="27" rot="R90"/>
+</element>
+<element name="JP10" library="pinhead" library_urn="urn:adsk.eagle:library:325" package="1X04" package3d_urn="urn:adsk.eagle:package:22407/2" value="" x="5.08" y="-158.75" smashed="yes">
+<attribute name="NAME" x="-0.0762" y="-156.9212" size="1.27" layer="25" ratio="10"/>
+<attribute name="POPULARITY" value="91" x="5.08" y="-158.75" size="1.778" layer="27" display="off"/>
+<attribute name="VALUE" x="0" y="-161.925" size="1.27" layer="27"/>
 </element>
 </elements>
@@
 <vertex x="0" y="0"/>
 </polygon>
-<contactref element="JP5" pad="3"/>
-<contactref element="JP4" pad="3"/>
-<contactref element="JP2" pad="3"/>
-<contactref element="R1" pad="1"/>
-<contactref element="JP2" pad="2"/>
-<contactref element="JP4" pad="2"/>
-<contactref element="JP5" pad="2"/>
-<contactref element="DC_IN" pad="2"/>
-<contactref element="U$1" pad="2"/>
-<contactref element="R4" pad="2"/>
-<contactref element="C3" pad="2"/>
-<contactref element="C2" pad="-"/>
-<wire x1="11.43" y1="59.27" x2="11.01" y2="59.69" width="0.6096" layer="1"/>
-<wire x1="9.74" y1="59.69" x2="11.01" y2="59.69" width="0.6096" layer="1"/>
-<wire x1="11.43" y1="59.27" x2="11.43" y2="54.61" width="0.6096" layer="1"/>
-<wire x1="27.52" y1="50.38" x2="27.68" y2="50.96" width="0.6096" layer="1"/>
-<wire x1="38.81" y1="17.78" x2="40.64" y2="17.78" width="0.4064" layer="1"/>
-<contactref element="JP1" pad="2"/>
-<contactref element="JP1" pad="3"/>
-<contactref element="JP3" pad="3"/>
-<contactref element="JP3" pad="2"/>
-<contactref element="R2" pad="1"/>
-<contactref element="Q2" pad="2"/>
-</signal>
-<signal name="+3V3">
-<contactref element="JP2" pad="1"/>
-<contactref element="JP4" pad="1"/>
-<contactref element="JP5" pad="1"/>
-<wire x1="6.35" y1="48.26" x2="6.35" y2="54.61" width="0.6096" layer="16"/>
-<contactref element="R1" pad="2"/>
-<wire x1="6.77" y1="59.69" x2="6.35" y2="59.27" width="0.6096" layer="1"/>
-<wire x1="6.35" y1="59.27" x2="6.35" y2="54.61" width="0.6096" layer="1"/>
-<wire x1="6.77" y1="59.69" x2="8.04" y2="59.69" width="0.6096" layer="1"/>
-<wire x1="6.35" y1="16.51" x2="6.35" y2="39.37" width="0.6096" layer="1"/>
-<wire x1="6.35" y1="39.37" x2="6.35" y2="48.26" width="0.6096" layer="1"/>
-<contactref element="JP1" pad="1"/>
-<contactref element="JP3" pad="1"/>
-<wire x1="6.35" y1="39.37" x2="6.35" y2="31.75" width="0" layer="19" extent="1-1"/>
-<wire x1="6.35" y1="15.24" x2="6.35" y2="16.51" width="0" layer="19" extent="1-1"/>
 </signal>
 <signal name="12V">
 <contactref element="K2" pad="1"/>
-<contactref element="D3" pad="C"/>
-<contactref element="DC_IN" pad="1"/>
-<contactref element="FAN_OUT" pad="1"/>
-<contactref element="D2" pad="C"/>
-<contactref element="C3" pad="1"/>
-<contactref element="C2" pad="+"/>
-<wire x1="34.78" y1="29.21" x2="34.85" y2="29.14" width="1.27" layer="1"/>
-<wire x1="34.85" y1="29.14" x2="34.85" y2="17.78" width="1.27" layer="1"/>
-<wire x1="34.78" y1="29.21" x2="34.78" y2="35.56" width="1.27" layer="1"/>
-<wire x1="34.78" y1="35.56" x2="34.78" y2="67.3258" width="1.27" layer="1"/>
-<wire x1="37.25" y1="35.56" x2="34.78" y2="35.56" width="0.6096" layer="1"/>
-<wire x1="28.4458" y1="73.66" x2="28.4458" y2="82.3458" width="1.27" layer="1"/>
-<wire x1="28.4458" y1="82.3458" x2="28.65" y2="82.55" width="1.27" layer="1"/>
-<wire x1="34.78" y1="67.3258" x2="28.4458" y2="73.66" width="1.27" layer="1"/>
-<contactref element="K1" pad="2"/>
-<contactref element="D1" pad="C"/>
-<contactref element="RELE_OUT1" pad="1"/>
-<contactref element="JP7" pad="2"/>
-<wire x1="95.25" y1="69.85" x2="81.99" y2="90.17" width="0" layer="19" extent="1-1"/>
-<wire x1="89.82" y1="62.96" x2="95.25" y2="69.85" width="0" layer="19" extent="1-1"/>
-<wire x1="82.16" y1="48.26" x2="89.82" y2="62.96" width="0" layer="19" extent="1-1"/>
-<wire x1="62.62" y1="50.8" x2="82.16" y2="48.26" width="0" layer="19" extent="1-1"/>
-<wire x1="62.23" y1="60.96" x2="62.62" y2="50.8" width="0" layer="19" extent="1-1"/>
-<wire x1="37.25" y1="35.56" x2="62.23" y2="60.96" width="0" layer="19" extent="1-1"/>
-</signal>
-<signal name="N$2">
-<contactref element="FAN_OUT" pad="2"/>
-<contactref element="U$1" pad="3"/>
-<contactref element="D2" pad="A"/>
-<wire x1="24.69" y1="82.55" x2="24.69" y2="73.66" width="1.27" layer="1"/>
-<wire x1="24.69" y1="73.66" x2="24.8942" y2="73.66" width="1.27" layer="1"/>
-<wire x1="25.4" y1="62.19" x2="24.8942" y2="62.6958" width="1.27" layer="1"/>
-<wire x1="24.8942" y1="73.66" x2="24.8942" y2="62.6958" width="1.27" layer="1"/>
-</signal>
-<signal name="N$3">
-<contactref element="R3" pad="1"/>
-<contactref element="R4" pad="1"/>
-<contactref element="U$1" pad="1"/>
-<wire x1="23.12" y1="54.89" x2="21.59" y2="53.08" width="0.6096" layer="1"/>
-<wire x1="21.59" y1="50.38" x2="21.59" y2="53.08" width="0.6096" layer="1"/>
-<wire x1="25.82" y1="50.38" x2="21.59" y2="50.38" width="0.6096" layer="1"/>
-</signal>
-<signal name="N$6">
-<contactref element="R3" pad="2"/>
 </signal>
 <signal name="N$1">
@@
 </signal>
 <signal name="N$11">
-<contactref element="Q1" pad="3"/>
 <contactref element="R6" pad="2"/>
-<wire x1="57.47" y1="44.45" x2="56.896" y2="49.8094" width="0" layer="19" extent="1-1"/>
+</signal>
+<signal name="N$21">
+<contactref element="JP1" pad="2"/>
+<contactref element="JP2" pad="2"/>
+<contactref element="JP4" pad="2"/>
+<contactref element="JP3" pad="2"/>
+<contactref element="JP5" pad="2"/>
+<wire x1="8.89" y1="48.26" x2="8.89" y2="54.61" width="0" layer="19" extent="1-1"/>
+<wire x1="8.89" y1="39.37" x2="8.89" y2="48.26" width="0" layer="19" extent="1-1"/>
+<wire x1="8.89" y1="31.75" x2="8.89" y2="39.37" width="0" layer="19" extent="1-1"/>
+<wire x1="8.89" y1="15.24" x2="8.89" y2="31.75" width="0" layer="19" extent="1-1"/>
+</signal>
+<signal name="N$22">
+<contactref element="JP2" pad="1"/>
+<contactref element="JP1" pad="1"/>
+<contactref element="JP4" pad="1"/>
+<contactref element="JP3" pad="1"/>
+<contactref element="JP5" pad="1"/>
+<wire x1="6.35" y1="48.26" x2="6.35" y2="54.61" width="0" layer="19" extent="1-1"/>
+<wire x1="6.35" y1="39.37" x2="6.35" y2="48.26" width="0" layer="19" extent="1-1"/>
+<wire x1="6.35" y1="31.75" x2="6.35" y2="39.37" width="0" layer="19" extent="1-1"/>
+<wire x1="6.35" y1="15.24" x2="6.35" y2="31.75" width="0" layer="19" extent="1-1"/>
+</signal>
+<signal name="N$3">
+</signal>
+<signal name="N$6">
+<contactref element="Q2" pad="3"/>
 </signal>
 <signal name="N$12">
-<contactref element="JP6" pad="4"/>
-<contactref element="R6" pad="1"/>
-<wire x1="59.69" y1="8.89" x2="59.37" y2="44.45" width="0" layer="19" extent="1-1"/>
+<contactref element="K1" pad="5"/>
 </signal>
-<signal name="N$13">
-<contactref element="JP6" pad="3"/>
-<contactref element="R7" pad="1"/>
-<wire x1="62.23" y1="8.89" x2="71.12" y2="39.69" width="0" layer="19" extent="1-1"/>
-</signal>
-<signal name="N$14">
-<contactref element="Q2" pad="3"/>
-<contactref element="R7" pad="2"/>
-<contactref element="R2" pad="2"/>
-<wire x1="71.12" y1="41.59" x2="76.454" y2="41.6306" width="0" layer="19" extent="1-1"/>
-<wire x1="71.44" y1="35.56" x2="71.12" y2="41.59" width="0" layer="19" extent="1-1"/>
-</signal>
-<signal name="N$15">
-<contactref element="D3" pad="A"/>
-</signal>
-<signal name="N$10">
-<contactref element="Q1" pad="1"/>
-<contactref element="K2" pad="16"/>
-<wire x1="54.864" y1="50.7746" x2="54.61" y2="60.96" width="0" layer="19" extent="1-1"/>
-</signal>
-<signal name="N$9">
-<contactref element="Q2" pad="1"/>
-<contactref element="K1" pad="5"/>
-<contactref element="D1" pad="A"/>
-<wire x1="77.86" y1="48.26" x2="77.82" y2="62.96" width="0" layer="19" extent="1-1"/>
-<wire x1="78.486" y1="40.6654" x2="77.86" y2="48.26" width="0" layer="19" extent="1-1"/>
-</signal>
-<signal name="N$17">
-<contactref element="JP7" pad="1"/>
-<contactref element="K1" pad="3"/>
-<wire x1="89.82" y1="75.16" x2="95.25" y2="72.39" width="0" layer="19" extent="1-1"/>
-</signal>
-<signal name="N$18">
-<contactref element="RELE_OUT1" pad="2"/>
-<contactref element="K1" pad="1"/>
-<wire x1="83.82" y1="60.96" x2="78.03" y2="90.17" width="0" layer="19" extent="1-1"/>
-</signal>
-<signal name="N$16">
-<contactref element="JP8" pad="2"/>
-<contactref element="RELE_OUT3" pad="1"/>
-<contactref element="K2" pad="4"/>
-<wire x1="3.81" y1="-135.89" x2="4.37" y2="-149.86" width="0" layer="19" extent="1-1"/>
-<wire x1="62.23" y1="68.58" x2="3.81" y2="-135.89" width="0" layer="19" extent="1-1"/>
-</signal>
-<signal name="N$19">
-<contactref element="JP9" pad="1"/>
-<contactref element="RELE_OUT2" pad="2"/>
-<wire x1="89.61" y1="24.13" x2="1.27" y2="-142.24" width="0" layer="19" extent="1-1"/>
-</signal>
-<signal name="N$20">
-<contactref element="JP9" pad="2"/>
-<contactref element="K2" pad="13"/>
-<wire x1="54.61" y1="68.58" x2="3.81" y2="-142.24" width="0" layer="19" extent="1-1"/>
+<signal name="N$2">
+<contactref element="JP3" pad="3"/>
+<contactref element="JP5" pad="3"/>
+<contactref element="JP4" pad="3"/>
+<contactref element="JP2" pad="3"/>
+<contactref element="JP1" pad="3"/>
+<wire x1="11.43" y1="48.26" x2="11.43" y2="54.61" width="0" layer="19" extent="1-1"/>
+<wire x1="11.43" y1="39.37" x2="11.43" y2="48.26" width="0" layer="19" extent="1-1"/>
+<wire x1="11.43" y1="31.75" x2="11.43" y2="39.37" width="0" layer="19" extent="1-1"/>
+<wire x1="11.43" y1="15.24" x2="11.43" y2="31.75" width="0" layer="19" extent="1-1"/>
 </signal>
 </signals>
