File: pcb/p4_joint.sch (EAGLE design)
At the start: 14 parts

Commit message: pcb(p4_joint): avance rev B (WIP, sin terminar)
Trabajo en curso del diseno: rele G5V-2, diodo SS14, transistores SOT-23 y
conectores 1X04 anadidos al esquema y la placa. Falta acabar el enrutado y la
revision final; se commitea para poder cortar el release v1.0.10 del firmware
con el arbol limpio.

Co-Authored-By: Claude Opus 4.8 (1M context) <noreply@anthropic.com>
Parts:
- added D1, D3: SS14, p4_joint_add:SS14
- added JP6: (no value), pinhead:PINHD-1X4
- added JP7, JP8, JP9: (no value), pinhead:PINHD-1X2
- added K1: JS1APF-B-12V, p4_joint_add:JS1APF-B-12V
- added K2: G5V-2, relay:G5V-2
- added Q1, Q2: 2N7002, zetex:NMOSSOT23
- added R2, R5: 10k, eagle-ltspice:R
- added R6, R7: 100, eagle-ltspice:R
- added RELE_OUT, RELE_OUT1, RELE_OUT2, RELE_OUT3: (no value), con-molex:KK-156-2
- JP1: value (none) -> DS18B20_IN; device pinhead:PINHD-1X2 -> pinhead:PINHD-1X3
- JP3: value DS18B20_1 -> DS18B20_3
- U$1: value IRLR7843 -> LR7843; LCSC (none) -> C9900160403
Connections:
- removed net DATA_DS18B20: JP2.3, JP3.3, JP4.3, JP5.3, R1.1
- new net N$10: K2A.2, Q1.D
- new net N$11: Q1.G, R6.2
- new net N$12: JP6.4, R6.1
- new net N$13: JP6.3, R7.1
- new net N$14: Q2.G, R2.2, R7.2
- new net N$15: D3.A
- new net N$16: JP8.2, K21.P, RELE_OUT3-1.S
- new net N$17: JP7.1, K1.NO
- new net N$18: K1.COM, RELE_OUT1-2.S
- new net N$19: JP9.1, RELE_OUT2-2.S
- new net N$20: JP9.2, K22.P
- new net N$5: R5.2
- new net N$9: D1.A, K1.C2, Q2.D
- net +3V3: now also JP1.1
- net 12V: now also D1.C, D3.C, JP7.2, K1.C1, K2A.1, RELE_OUT1-1.S
- net GND: now also JP1.2, JP1.3, JP2.3, JP3.3, JP4.3, JP5.3, Q2.S, R1.1, R2.1
- net N$6: no longer JP1.1
