File: pcb/p4_joint.sch (EAGLE design)
At the start: 32 parts, among them K1 JS1APF-B-12V, K2 G5V-2, Q1 2N7002, Q2 2N7002

Commit message: fix(ne185): filtrar el baile del nivel de agua limpia segun si el motor esta en marcha
Parts:
- added JP10: (no value), pinhead:PINHD-1X4
Connections:
- removed net +3V3: JP1.1, JP2.1, JP3.1, JP4.1, JP5.1, R1.2
- removed net GND: C2.-, C3.2, DC_IN-2.S, JP1.2, JP1.3, JP2.2, JP2.3, JP3.2, JP3.3, JP4.2, JP4.3, JP5.2, JP5.3, Q2.S, R1.1, R2.1, R4.2, U$1.S
- removed net N$10: K2A.2, Q1.D
- removed net N$13: JP6.3, R7.1
- removed net N$14: Q2.G, R2.2, R7.2
- removed net N$15: D3.A
- removed net N$16: JP8.2, K21.P, RELE_OUT3-1.S
- removed net N$17: JP7.1, K1.NO
- removed net N$18: K1.COM, RELE_OUT1-2.S
- removed net N$19: JP9.1, RELE_OUT2-2.S
- removed net N$20: JP9.2, K22.P
- removed net N$3: R3.1, R4.1, U$1.G
- removed net N$9: D1.A, K1.C2, Q2.D
- new net N$21: JP1.2, JP2.2, JP3.2, JP4.2, JP5.2
- new net N$22: JP1.1, JP2.1, JP3.1, JP4.1, JP5.1
- net 12V: no longer C2.+, C3.1, D1.C, D2.12, D3.C, DC_IN-1.S, FAN_OUT-1.S, JP7.2, K1.C1, RELE_OUT1-1.S
- net N$11: no longer Q1.G
- net N$12: now also K1.C2; no longer JP6.4, R6.1
- net N$2: now also JP1.3, JP2.3, JP3.3, JP4.3, JP5.3; no longer D2.21, FAN_OUT-2.S, U$1.D
- net N$6: now also Q2.G; no longer R3.2
